File: Potentiostat KiCAD Prohject/Potentiostat KiCAD Prohject.kicad_sch (KiCad schematic)
At the start: 51 parts, among them J1 Conn_01x02_Pin, J2 USB_C_Receptacle_USB2.0, J3 Conn_01x02_Pin, J4 Reference Electrode, J5 Working Electrode, J6 Working Electrode, K1 DIPxx-1Axx-12xD, SW1 Reset, SW2 Boot, U1 OPA2277, U10 ADS1115IDGS, U11 MCP4725xxx-xCH, U13 LD1117S33TR_SOT223, U14 ESP32-S2-SOLO, U2 TL074, U4 OPA2277, U5 INA128, U6 MCP4725xxx-xCH, U7 INA128, U8 REF3033, U9 INA128

Commit message: finished!
Parts:
- added H1, H2, H3, H4: MountingHole_Pad, symbol Mechanical:MountingHole_Pad
- added TP1, TP10, TP11, TP12, TP13, TP14, TP15, TP16, TP17, TP18, TP19, TP2, TP20, TP21, TP22, TP23, TP24, TP25, TP26, TP3, TP4, TP5, TP6, TP7, TP8, TP9: TestPoint, TestPoint:TestPoint_Pad_1.0x1.0mm, symbol Connector:TestPoint
Connections:
- net +5V: now also TP9.1
- net +9V: now also TP4.1
- net -9V: now also TP2.1
- net ADC_IN3: now also TP20.1
- net GND: now also H1.1, H2.1, H3.1, H4.1, TP3.1
- net I2C_SCL: now also TP10.1, TP6.1, TP7.1
- net I2C_SDA: now also TP11.1, TP5.1, TP8.1
- net at R17.2, R4.2, R8.1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: now also TP22.1
- net at J6.1 (Pin_1), U5.2 (-): now also TP1.1
- net at R15.1, R16.2, R2.2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: now also TP23.1
- net at R13.2, R14.1, R15.2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: now also TP24.1
- net at D2.1 (K), U10.6 (AIN2), U9.2 (-)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: now also TP26.1
- net at R5.1, U11.1 (VOUT): now also TP21.1
- net at J5.1 (Pin_1), K1.13, K1.2: now also TP13.1
- net at C1.2, R10.2, R11.1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: now also TP14.1
- net at J4.1 (Pin_1), U2.12 (+): now also TP12.1
- net at R13.1, R14.2, U7.6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: now also TP25.1
- net at K1.6, U4.1: now also TP16.1
- net at U4.3 (+), U8.2 (OUT): now also TP15.1
- net at R6.2, R7.2, R8.2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: now also TP17.1
- net at U1.6 (-), U6.1 (VOUT): now also TP19.1
- net at R10.1, R9.2, U2.1: now also TP18.1
